Commit message: Added Robosub 2019 code

File: uuv_descriptions/urdf/rexrov_sensors.xacro (robot description, xacro)
@@ -39,11 +39,14 @@
   <!-- Mount a camera -->
   <xacro:default_camera namespace="${namespace}" parent_link="${namespace}/base_link" suffix="">
-    <origin xyz="1.15 0 0.4" rpy="0 0.6 0"/>
+    <origin xyz="1.15 0 0.4" rpy="0 0 0"/>
   </xacro:default_camera>
   <xacro:default_camera namespace="${namespace}" parent_link="${namespace}/base_link" suffix="right">
-    <origin xyz="1.15 -0.63 0.4" rpy="0 0.6 0.4"/>
+    <origin xyz="1.15 -0.63 0.4" rpy="0 0 0"/>
   </xacro:default_camera>
   <xacro:default_camera namespace="${namespace}" parent_link="${namespace}/base_link" suffix="left">
-    <origin xyz="1.15 0.63 0.4" rpy="0 0.6 -0.4"/>
+    <origin xyz="1.15 0.63 0.4" rpy="0 0 0"/>
+  </xacro:default_camera>
+  <xacro:default_camera namespace="${namespace}" parent_link="${namespace}/base_link" suffix="down">
+    <origin xyz="1.15 0 -0.8" rpy="0 1.5708 0"/>
   </xacro:default_camera>
   <!-- Mount a GPS. -->
